Commit message: cleanup

File: my_robot/urdf/r2-d2.xacro (robot description, xacro)
@@ -20,5 +20,4 @@
         <cylinder radius="0.2" length="0.6"/>
       </geometry>
-      <material name="blue"/>
     </visual>
     <collision>
@@ -42,5 +41,4 @@
           <cylinder radius="${wheeldiam/2}" length="0.1"/>
         </geometry>
-        <material name="black"/>
       </visual>
       <collision>
@@ -66,5 +64,4 @@
         </geometry>
         <origin xyz="0 0 -${leglen/2}" rpy="0 ${pi/2} 0"/>
-        <material name="white"/>
       </visual>
       <collision>
@@ -86,5 +83,4 @@
           <box size="${baselen} 0.1 0.1"/>
         </geometry>
-        <material name="white"/>
       </visual>
       <collision>
@@ -110,5 +106,4 @@
         <sphere radius="0.2"/>
       </geometry>
-      <material name="white"/>
     </visual>
     <collision>
